Commit message: in the humble container, enabled  ros2 launch iiwa_description display_iiwa.launch.py

File: colcon_ws/src/iiwa_description/urdf/iiwa14_description.xacro (robot description, xacro)
@@ -4,7 +4,8 @@
     <xacro:macro name="iiwa14"
         params="robot_name:=^|lbr mode:=^|mock">
+        <xacro:arg name="system_config_path" default="$(find iiwa_description)/ros2_control/lbr_system_config.yaml" />
         <!-- joint limits via yaml -->
         <xacro:property name="joint_limits_path"
-            value="$(find iiwa_description)/urdf/iiwa14/joint_limits.yaml" />
+            value="$(find iiwa_description)/urdf/joint_limits.yaml" />
         <xacro:property name="joint_limits" value="${xacro.load_yaml(joint_limits_path)}" />
         <!-- constants -->
@@ -12,4 +13,9 @@
         <xacro:property name="joint_damping" value="10.0" />
         <xacro:property name="joint_friction" value="0.1" />
+        <xacro:iiwa_gripper_system_interface
+            robot_name="${robot_name}"
+            mode="${mode}"
+            joint_limits="${joint_limits}"
+            system_config_path="$(arg system_config_path)" />
         <link name="${robot_name}_link_0">
             <inertial>
@@ -286,76 +292,11 @@
         <link name="${robot_name}_link_ee">
         </link>
-    <link name="tool_mount">
-        <visual>
-            <origin xyz="0 0 0" rpy="0 ${-pi/2} ${pi/2}"/>
-            <geometry>
-                <mesh filename="package://iiwa_description/meshes/envs/visual/iiwa_tool_mount.stl"/>
-            </geometry>
-            <material name="">
-                <color rgba="0.8 0.8 0.8 1"/>
-            </material>
-        </visual>
-        <collision>
-            <origin xyz="0 0 0.005" rpy="0 0 0"/>
-            <geometry>
-                <cylinder length="0.006" radius="0.038"/>
-            </geometry>
-        </collision>
-    </link>
-    <joint name="eef_base_joint" type="fixed">
-        <origin xyz="0 0 0.0095" rpy="0 0 0"/>
-        <parent link="tool_mount"/>
-        <child link="eef_base"/>
-    </joint>
-    <link name="eef_base">
-        <visual>
-            <origin xyz="0 0 0" rpy="0 0 0"/>
-            <geometry>
-                <mesh filename="package://iiwa_description/meshes/envs/visual/hande_base.stl"/>
-            </geometry>
-            <material name="">
-                <color rgba="0.8 0.8 0.8 1"/>
-            </material>
-        </visual>
-        <collision>
-            <origin xyz="0 0 0.0095" rpy="0 0 0"/>
-            <geometry>
-                <cylinder length="0.020" radius="0.038"/>
-            </geometry>
-        </collision>
-    </link>
-    <joint name="eef_joint" type="fixed">
-        <origin xyz="0 0 0.0015" rpy="0 0 3.14"/>
-        <parent link="eef_base"/>
-        <child link="eef"/>
-    </joint>
-    <link name="eef">
-        <visual>
-            <origin xyz="0 0 0" rpy="0 0 0"/>
-            <geometry>
-                <mesh filename="package://iiwa_description/meshes/envs/visual/hande.stl"/>
-            </geometry>
-            <material name="">
-                <color rgba="0.8 0.8 0.8 1"/>
-            </material>
-        </visual>
-        <collision>
-            <geometry>
-                <mesh filename="package://iiwa_description/meshes/envs/collision/hande.stl"/>
-            </geometry>
-        </collision>
-    </link>
-    <joint name="tool_joint" type="fixed">
-        <parent link="${robot_name}_link_ee"/>
-        <child link="tool_mount"/>
-        <origin xyz="0 0 0.001" rpy="0 0 ${PI/2}"/>
-    </joint>
-    <joint name="tool_tip_joint" type="fixed">
-        <parent link="${robot_name}_link_ee"/>
-        <child link="tool_link_ee"/>
-        <origin xyz="0 0 0.25" rpy="${PI/2} -${PI/2} 0"/>
-    </joint>
-    <!--  The TCP frame is here defined -->
-    <link name="tool_link_ee"/>
+        <!--  The TCP frame is here defined -->
+        <link name="tool_link_ee"/>
+        <joint name="tool_tip_joint" type="fixed">
+            <parent link="${robot_name}_link_ee"/>
+            <child link="tool_link_ee"/>
+            <origin xyz="0 0 0.25" rpy="${PI/2} -${PI/2} 0"/>
+        </joint>
     </xacro:macro>
 </robot>

File: colcon_ws/src/iiwa_description/urdf/iiwa14_rq140.xacro (robot description, xacro)
@@ -3,5 +3,5 @@
 <robot name="iiwa_gripper" xmlns:xacro="http://www.ros.org/wiki/xacro">
     <!-- include the lbr iiwa macro -->
-    <xacro:include filename="$(find iiwa_description)/urdf/iiwa14/iiwa14_description.xacro" />
+    <xacro:include filename="$(find iiwa_description)/urdf/iiwa14_description.xacro" />
     <xacro:include filename="$(find iiwa_description)/urdf/robotiq_arg2f_140_model_macro.xacro" />
     <xacro:include filename="$(find iiwa_description)/gazebo/iiwa_gripper_gazebo.xacro" />
@@ -9,12 +9,6 @@
     <xacro:arg name="robot_name" default="lbr" />
     <xacro:arg name="mode" default="true" />
-    <xacro:arg name="system_config_path" default="$(find iiwa_description)/ros2_control/lbr_system_config.yaml" />
     <!-- macros for gazebo / mock / hardware -->
-    <xacro:lbr_gazebo robot_name="${robot_name}" />
-    <xacro:iiwa_gripper_system_interface
-        robot_name="${robot_name}"
-        mode="${mode}"
-        joint_limits="${joint_limits}"
-        system_config_path="${system_config_path}" />
+    <xacro:lbr_gazebo robot_name="$(arg robot_name)" />
 	<link name="world" />
 	<link name="base_link"/>
@@ -24,29 +18,7 @@
 		<origin xyz="0.0 0.0 0.0" rpy="0.0 0.0 0.0" />
 	</joint>
-    <link name="workspace_mount1">
-        <visual>
-            <origin xyz="0 0 0" rpy="0 0 0"/>
-            <geometry>
-                <box size="0.3 0.3 0.03"/>
-            </geometry>
-            <material name="gray">
-                <color rgba="0.7 0.7 0.7 0.2"/>
-            </material>
-        </visual>
-        <collision>
-            <origin xyz="0 0 0" rpy="0 0 0"/>
-            <geometry>
-                <box size="0.3 0.3 0.03"/>
-            </geometry>
-        </collision>
-    </link>
-    <joint name="workspace_mount1_joint" type="fixed">
-        <origin xyz="0.1 0.5 0.85" rpy="0 0 3.14"/>
-        <parent link="base_link"/>
-        <child link="workspace_mount1"/>
-    </joint>
-    <joint name="$(arg robot_name)_joint" type="fixed">
-        <origin xyz="0 0 0.016" rpy="0 0 2.36"/>
-        <parent link="workspace_mount1" />
+    <joint name="world_$(arg robot_name)_joint" type="fixed">
+        <origin xyz="0 0 0" rpy="0 0 0"/>
+        <parent link="world" />
         <child link="$(arg robot_name)_link_0" />
     </joint>
@@ -57,5 +29,5 @@
 	<xacro:robotiq_arg2f_140 prefix="" />
 	<joint name="iiwa_ee_link_gripper_base" type="fixed">
-		<parent link="tool_link_ee" />
+		<parent link="lbr_link_ee" />
 		<child link="robotiq_arg2f_base_link" />
 		<origin xyz="0.0 0.0 0.0" rpy="0.0 0.0 ${pi/2}" />
