Commit message: add mujoco env

File: dataset/urdfs/iiwa14_rq140.urdf (robot description, URDF)
Before this commit: robot iiwa_gripper, 23 links, 22 joints
Joints:
- joint iiwa_joint_2: origin xyz=0 0 0.2025 rpy=1.5707963267948966   0 3.141592653589793 -> xyz=0 0 0.2025 rpy=1.5707963267948966 0 3.141592653589793
