Commit message: fix bugs

File: dataset/urdfs/iiwa14_rqhe.urdf (robot description, URDF)
Before this commit: robot iiwa_gripper, 18 links, 17 joints
Links:
- link hand_e_link: geometry collision mesh filename=/dataset/meshes/hande/hande.stl scale=1.0 1.0 1.0; visual mesh filename=/dataset/meshes/hande/hande.stl scale=1.0 1.0 1.0
- link hande_left_finger: geometry collision mesh filename=/dataset/meshes/hande/finger_1.stl scale=1.0 1.0 1.0; visual mesh filename=/dataset/meshes/hande/finger_1.stl scale=1.0 1.0 1.0
- link hande_right_finger: geometry collision mesh filename=/dataset/meshes/hande/finger_2.stl scale=1.0 1.0 1.0; visual mesh filename=/dataset/meshes/hande/finger_2.stl scale=1.0 1.0 1.0

File: dataset/urdfs/iiwa14_rqhe_sdf.urdf (robot description, URDF)
Before this commit: robot iiwa_gripper, 18 links, 17 joints
Links:
- link hand_e_link: geometry collision mesh filename=/dataset/meshes/hande/hande.stl scale=1.0 1.0 1.0; visual mesh filename=/dataset/meshes/hande/hande.stl scale=1.0 1.0 1.0
- link hande_left_finger: geometry collision mesh filename=/dataset/meshes/hande/finger_1.stl scale=1.0 1.0 1.0; visual mesh filename=/dataset/meshes/hande/finger_1.stl scale=1.0 1.0 1.0
- link hande_right_finger: geometry collision mesh filename=/dataset/meshes/hande/finger_2.stl scale=1.0 1.0 1.0; visual mesh filename=/dataset/meshes/hande/finger_2.stl scale=1.0 1.0 1.0
