Commit message: add gazebo simulation env and update README

File: catkin_ws/src/iiwa_description/urdf/iiwa.gazebo.xacro (robot description, xacro)
@@ -56,4 +56,30 @@
       <mu2>0.2</mu2>
     </gazebo>
+    <gazebo reference="iiwa_joint_1">
+        <implicitSpringDamper>True</implicitSpringDamper>
+    </gazebo>
+    <gazebo reference="iiwa_joint_2">
+        <implicitSpringDamper>True</implicitSpringDamper>
+    </gazebo>
+    <gazebo reference="iiwa_joint_3">
+        <implicitSpringDamper>True</implicitSpringDamper>
+    </gazebo>
+    <gazebo reference="iiwa_joint_4">
+        <implicitSpringDamper>True</implicitSpringDamper>
+    </gazebo>
+    <gazebo reference="iiwa_joint_5">
+        <implicitSpringDamper>True</implicitSpringDamper>
+    </gazebo>
+    <gazebo reference="iiwa_joint_6">
+        <implicitSpringDamper>True</implicitSpringDamper>
+    </gazebo>
+    <gazebo reference="iiwa_joint_7">
+        <implicitSpringDamper>True</implicitSpringDamper>
+    </gazebo>
+    <gazebo>
+        <plugin filename="libgazebo_ros_control.so" name="gazebo_ros_control">
+            <parameters>$(find iiwa_moveit_config)/config/gazebo_controllers.yaml</parameters>
+        </plugin>
+    </gazebo>
   </xacro:macro>
 </robot>

File: catkin_ws/src/iiwa_description/urdf/iiwa14.xacro (robot description, xacro)
@@ -3,6 +3,4 @@
   <!-- Import all Gazebo-customization elements, including Gazebo colors -->
   <xacro:include filename="$(find iiwa_description)/urdf/iiwa.gazebo.xacro" />
-  <!-- Import Transmissions -->
-  <xacro:include filename="$(find iiwa_description)/urdf/iiwa.transmission.xacro" />
   <!-- Include Utilities -->
   <xacro:include filename="$(find iiwa_description)/urdf/utilities.xacro" />
@@ -303,5 +301,74 @@
     <!--Extensions -->
     <xacro:iiwa_gazebo robot_name="${robot_name}" />
-    <xacro:iiwa_transmission hardware_interface="${hardware_interface}"/>
+    <transmission name="trans_iiwa_joint_1">
+        <type>transmission_interface/SimpleTransmission</type>
+        <joint name="iiwa_joint_1">
+            <hardwareInterface>hardware_interface/EffortJointInterface</hardwareInterface>
+        </joint>
+        <actuator name="iiwa_joint_1_motor">
+            <hardwareInterface>hardware_interface/EffortJointInterface</hardwareInterface>
+            <mechanicalReduction>1</mechanicalReduction>
+        </actuator>
+    </transmission>
+    <transmission name="trans_iiwa_joint_2">
+        <type>transmission_interface/SimpleTransmission</type>
+        <joint name="iiwa_joint_2">
+            <hardwareInterface>hardware_interface/EffortJointInterface</hardwareInterface>
+        </joint>
+        <actuator name="iiwa_joint_2_motor">
+            <hardwareInterface>hardware_interface/EffortJointInterface</hardwareInterface>
+            <mechanicalReduction>1</mechanicalReduction>
+        </actuator>
+    </transmission>
+    <transmission name="trans_iiwa_joint_3">
+        <type>transmission_interface/SimpleTransmission</type>
+        <joint name="iiwa_joint_3">
+            <hardwareInterface>hardware_interface/EffortJointInterface</hardwareInterface>
+        </joint>
+        <actuator name="iiwa_joint_3_motor">
+            <hardwareInterface>hardware_interface/EffortJointInterface</hardwareInterface>
+            <mechanicalReduction>1</mechanicalReduction>
+        </actuator>
+    </transmission>
+    <transmission name="trans_iiwa_joint_4">
+        <type>transmission_interface/SimpleTransmission</type>
+        <joint name="iiwa_joint_4">
+            <hardwareInterface>hardware_interface/EffortJointInterface</hardwareInterface>
+        </joint>
+        <actuator name="iiwa_joint_4_motor">
+            <hardwareInterface>hardware_interface/EffortJointInterface</hardwareInterface>
+            <mechanicalReduction>1</mechanicalReduction>
+        </actuator>
+    </transmission>
+    <transmission name="trans_iiwa_joint_5">
+        <type>transmission_interface/SimpleTransmission</type>
+        <joint name="iiwa_joint_5">
+            <hardwareInterface>hardware_interface/EffortJointInterface</hardwareInterface>
+        </joint>
+        <actuator name="iiwa_joint_5_motor">
+            <hardwareInterface>hardware_interface/EffortJointInterface</hardwareInterface>
+            <mechanicalReduction>1</mechanicalReduction>
+        </actuator>
+    </transmission>
+    <transmission name="trans_iiwa_joint_6">
+        <type>transmission_interface/SimpleTransmission</type>
+        <joint name="iiwa_joint_6">
+            <hardwareInterface>hardware_interface/EffortJointInterface</hardwareInterface>
+        </joint>
+        <actuator name="iiwa_joint_6_motor">
+            <hardwareInterface>hardware_interface/EffortJointInterface</hardwareInterface>
+            <mechanicalReduction>1</mechanicalReduction>
+        </actuator>
+    </transmission>
+    <transmission name="trans_iiwa_joint_7">
+        <type>transmission_interface/SimpleTransmission</type>
+        <joint name="iiwa_joint_7">
+            <hardwareInterface>hardware_interface/EffortJointInterface</hardwareInterface>
+        </joint>
+        <actuator name="iiwa_joint_7_motor">
+            <hardwareInterface>hardware_interface/EffortJointInterface</hardwareInterface>
+            <mechanicalReduction>1</mechanicalReduction>
+        </actuator>
+    </transmission>
   </xacro:macro>
 </robot>
